Commit message: Fix: fix link of imu of urdf

File: models/if750a_fix_motor/if750a_fix_motor.urdf (robot description, URDF)
Before this commit: robot if750a_fix_motor, 8 links, 7 joints
Links:
- removed link /imu_link
- added link downward_camera_link, mass 0.015
- added link front_camera_link, mass 0.015
- added link imu_link, mass 0.015
- added link left_camera_link, mass 0.015
- added link right_camera_link, mass 0.015
Joints:
- removed joint /imu_joint
- added joint downward_camera_joint: type fixed, parent base_link, child downward_camera_link, origin xyz=0.127909 0 0.187349 rpy=0 1.570796327 0
- added joint front_camera_joint: type fixed, parent base_link, child front_camera_link, origin xyz=0.1358 0 0.2282 rpy=0 0.19198621771 0
- added joint imu_joint: type revolute, parent base_link, child imu_link, origin xyz=0 0 0, axis 1 0 0, limit lower=0 upper=0 effort=0 velocity=0
- added joint left_camera_joint: type fixed, parent base_link, child left_camera_link, origin xyz=0.085811 0.092407 0.210252 rpy=0 0.192440003 1.40964135
- added joint right_camera_joint: type fixed, parent base_link, child right_camera_link, origin xyz=0.085811 0.092407 0.210252 rpy=0 0.192440003 1.40964135

Commit message: Fix: fix camera position in urdf

File: models/if750a_fix_motor/if750a_fix_motor.urdf (robot description, URDF)
Before this commit: robot if750a_fix_motor, 12 links, 11 joints
Joints:
- joint downward_camera_joint: origin xyz=0.127909 0 0.187349 rpy=0 1.570796327 0 -> xyz=0.127909 0 0.187349 rpy=0 0.7853981635 0
- joint right_camera_joint: origin xyz=0.085811 0.092407 0.210252 rpy=0 0.192440003 1.40964135 -> xyz=0.085811 -0.092407 0.210252 rpy=0 0.192440003 -1.40964135

Commit message: Fixed: update camera position on if750a_wx200 for better PCS streaming

File: models/if750a_fix_motor/if750a_fix_motor.urdf (robot description, URDF)
Before this commit: robot if750a_fix_motor, 12 links, 11 joints
Joints:
- joint left_camera_joint: origin xyz=0.085811 0.092407 0.210252 rpy=0 0.192440003 1.40964135 -> xyz=0.085811 0.092407 0.210252 rpy=0 0.192440003 0.96
- joint right_camera_joint: origin xyz=0.085811 -0.092407 0.210252 rpy=0 0.192440003 -1.40964135 -> xyz=0.085811 -0.092407 0.210252 rpy=0 0.192440003 -0.96
