Commit message: Change camera pose

File: models/if750a_camera_pushing/if750a_camera_pushing.urdf (robot description, URDF)
Before this commit: robot if750a, 13 links, 12 joints
Joints:
- joint front_camera_joint: origin xyz=0.1358 0 0.2282 rpy=0 0.19198621771 0 -> xyz=0.14227 0 0.2282 rpy=0 0.366519143 0
- joint left_camera_joint: origin xyz=0.085811 0.092407 0.210252 rpy=0 0.192440003 1.40964135 -> xyz=0.09942 0.10153 0.2282 rpy=0 0.366519143 0.968657735
- joint right_camera_joint: origin xyz=0.085811 0.092407 0.210252 rpy=0 0.192440003 1.40964135 -> xyz=0.09942 -0.10153 0.2282 rpy=0 0.366519143 -0.968657735

Commit message: Feat: if750a vertical rod

File: models/if750a_camera_pushing/if750a_camera_pushing.urdf (robot description, URDF)
Before this commit: robot if750a, 13 links, 12 joints
Links:
- added link velodyne_link, mass 0.001; visual mesh filename=file:///opt/ros/melodic/share/velodyne_description/meshes/V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 scale=1 1 1; visual mesh filename=file:///opt/ros/melodic/share/velodyne_description/meshes/V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 scale=1 1 1
- added link vertical_rod_link, mass 0.001; visual cylinder length=0.25 radius=0.03
Joints:
- added joint velodyne_joint: type fixed, parent base_link, child velodyne_link, origin xyz=0 0 0.125 rpy=0 0 0
- added joint vertical_rod_joint: type prismatic, parent base_link, child vertical_rod_link, origin xyz=0 0 0.125 rpy=0 0 0, axis 0 0 1, limit lower=-0.5 upper=0.0 effort=0.5 velocity=0.15
- joint horizontal_rod_joint: origin xyz=0.0 0 0.0 rpy=0 0 0 -> xyz=0.0 0 0.05 rpy=0 0 0
